File: power_dist_board/pcb-v3.kicad_pcb (KiCad board)
At the start: 2 copper layers, 113 x 70 mm, 16 parts, among them J1 Screw_Terminal_01x02, J2 Conn_01x07_Socket, J3 Screw_Terminal_01x02, J4 Screw_Terminal_01x02, J5 Conn_02x20_Odd_Even

Commit message: Remap Jetson pins and update labels
Connections:
- C2 pad 1: GND -> +12V
- J5 pad 1: (no net) -> +3.3V
- J5 pad 17: (no net) -> +3.3V
- J5 pad 2: (no net) -> +5V
- J5 pad 27: unconnected-(J5-Pin_27-Pad27) -> SDA
- J5 pad 28: unconnected-(J5-Pin_28-Pad28) -> SCL
- J5 pad 3: SDA -> unconnected-(J5-Pin_3-Pad3)
- J5 pad 4: (no net) -> +5V
- J5 pad 5: SCL -> unconnected-(J5-Pin_5-Pad5)
Routing:
- net SCL: track 114.7 -> 191.0 mm
- net SDA: track 124.1 -> 133.7 mm
- net ESC: track 116.5 -> 121.1 mm
Other:
- copper layers 2 -> 4
- board text added: "5V"
- board text added: "GND"
- board text added: "SCL"
- board text added: "SDA"
- board text added: "SERV"

Commit message: 2025
Parts:
- removed the C2 at (181.0, 67.0)
- removed C3: CP_Radial_D6.3mm_P2.50mm, Capacitor_THT:CP_Radial_D6.3mm_P2.50mm
- removed J1: Screw_Terminal_01x02, Connector_PinHeader_2.54mm:PinHeader_1x02_P2.54mm_Horizontal
- moved J3 57.5 mm to (151.0, 86.0), turned to -90 degrees
- moved C1 42.4 mm to (142.0, 46.0), turned to 180 degrees
- moved U2 35.7 mm to (195.3, 90.1)
- moved ? 34.0 mm to (200.0, 94.0)
- moved ? 33.5 mm to (200.5, 31.0)
- moved J4 33.5 mm to (141.3, 86.1)
- moved J2 27.5 mm to (166.0, 70.6)
- moved Q1 27.4 mm to (137.3, 30.5), turned to 180 degrees
- moved Q2 27.2 mm to (146.1, 30.3), turned to -90 degrees
- moved C2 17.2 mm to (165.8, 43.0)
Connections:
- C1 pad 1: ESC -> +5V
- C2 pad 2: +12V -> GND
- J5 pad 2: +5V -> (no net)
- J5 pad 4: +5V -> (no net)
- Q1 pad 1: +12V -> STABLE_12V
Routing:
- net ESC: track 121.1 -> 45.8 mm
- net STABLE_12V: track 22.8 -> 57.4 mm
- net SCL: track 191.0 -> 164.4 mm
- net +5V: track 76.9 -> 51.0 mm
- net SDA: track 133.7 -> 112.8 mm
- net +12V: track 36.9 -> 22.9 mm
Other:
- board size 113 x 70 mm -> 79.5 x 70 mm
- board text added: "10"
- board text added: "12"
- board text added: "14"
- board text added: "16"
- board text added: "18"
- board text added: "2"
- board text added: "20"
- board text added: "22"
- board text added: "24"
- board text added: "26"
- board text added: "28"
- board text added: "30"
- board text added: "32"
- board text added: "34"
- board text added: "36"
- board text added: "38"
- board text added: "4"
- board text added: "40"
- board text added: "8"
- board text added: "Boost"
- board text added: "Buck"
- board text added: "GSR"
- board text removed: "Boost Converter (12v)"
- board text removed: "Buck Converter (12v-5v)"
